File: pcb/CERAM-V2.kicad_pcb (KiCad board)
At the start: 2 copper layers, 52.2 x 95.5 mm, 24 parts, among them J1 Screw_Terminal_01x02, J10 Screw_Terminal_01x02, J11 Screw_Terminal_01x02, J12 Conn_01x06_Pin, J2 Conn_01x03_Pin, J3 Conn_01x03_Pin, J4 Conn_01x03_Pin, J5 Conn_01x03_Pin, J6 Conn_01x08_Pin, J8 Conn_01x04_Pin, J9 Conn_01x04_Pin, Q1 IRLZ44N, Q2 IRLZ44N, U1 XIAO-ESP32-S3-DIP, U2 LM317_TO-220

Commit message: Routing fix + readme polish + images + firmware
Parts:
- moved J6 17.6 mm to (123.5, 73.2), turned to 180 degrees
Routing:
- net GND: track 220.0 -> 250.9 mm
- net PYRO1: track 29.6 -> 52.3 mm
- net 5V: track 113.2 -> 128.4 mm
- net SDA: track 84.3 -> 95.1 mm
- net PWM3: track 69.3 -> 79.6 mm
- net 3V3: track 112.1 -> 118.5 mm
- net Net-(J10-Pin_1): track 22.7 -> 28.0 mm
- net PYRO2: track 46.7 -> 50.1 mm
- net Net-(U2-ADJ): track 30.4 -> 32.7 mm
- net SCL: track 94.2 -> 94.8 mm, vias 0 -> 1

Commit message: silkscreen + moved xiao
Parts:
- moved U1 9.45 mm to (113.7, 32.3)
Routing:
- net PWM1: track 70.9 -> 93.8 mm
- net GND: track 250.9 -> 228.5 mm, vias 0 -> 4
- net SDA: track 95.1 -> 116.4 mm, vias 1 -> 0
- net SCL: track 94.8 -> 115.5 mm, vias 1 -> 3
- net PWM4: track 64.8 -> 79.2 mm
- net PWM3: track 79.6 -> 93.6 mm
- net 5V: track 128.4 -> 141.9 mm, vias 0 -> 2
- net PYRO1: track 52.3 -> 42.5 mm
- net PYRO2: track 50.1 -> 59.6 mm
- net PWM2: track 70.0 -> 77.7 mm
- net RX: track 29.8 -> 27.8 mm, vias 0 -> 1
- net 3V3: track 118.5 -> 116.5 mm, vias 0 -> 1
- net unconnected-(U1-GPIO7/D8/A8/SCK-Pad9): track 0.84 -> 0.00 mm
Other:
- board text added: "3v3 here"
- board text added: "BMP280 Here"
- board text added: "By Ahsan A"
- board text added: "CERAMv2"
- board text added: "I2C"
- board text added: "MPU6050 Here"
- board text added: "PWM Channels"
- board text added: "SOLDER WITH HEADERS ON"
- board text added: "UART"
- board text added: "VCC GND SCL SDA"
